File: src/pcbs/form-uno/form-uno.kicad_pcb (KiCad board)
At the start: 2 copper layers, 272.6 x 122.9 mm, 121 parts, among them SW1 SW_Push, SW10 SW_Push, SW11 SW_Push, SW12 SW_Push, SW13 SW_Push, SW14 SW_Push, SW15 SW_Push, SW16 SW_Push, SW17 SW_Push, SW18 SW_Push, SW19 SW_Push, SW2 SW_Push, SW20 SW_Push, SW21 SW_Push, SW22 SW_Push, SW23 SW_Push, SW24 SW_Push, SW25 SW_Push, SW26 SW_Push, SW27 SW_Push, SW28 SW_Push, SW29 SW_Push, SW3 SW_Push, SW30 SW_Push, SW31 SW_Push, SW32 SW_Push, SW33 SW_Push, SW34 SW_Push, SW35 SW_Push, SW36 SW_Push, SW37 SW_Push, SW38 SW_Push, SW39 SW_Push, SW4 SW_Push, SW40 SW_Push, SW41 SW_Push, SW42 SW_Push, SW43 SW_Push, SW44 SW_Push, SW45 SW_Push, SW46 SW_Push, SW47 SW_Push, SW48 SW_Push, SW49 SW_Push, SW5 SW_Push, SW50 SW_Push, SW51 SW_Push, SW52 SW_Push, SW53 SW_Push, SW54 SW_Push, SW55 SW_Push, SW56 SW_Push, SW57 SW_Push, SW58 SW_Push, SW59 SW_Push, SW6 SW_Push, SW60 SW_Push, SW7 SW_Push, SW8 SW_Push, SW9 SW_Push, U1 rp2040-zero

Commit message: Route the board matrix
Parts:
- moved SW42 2.01 mm to (123.4, 105.5)
- moved D10 2.01 mm to (220.7, 42.6)
- moved SW15 2.01 mm to (72.4, 57.4)
- moved SW29 2.01 mm to (107.5, 81.6)
- moved SW19 2.01 mm to (174.5, 67.7)
- moved SW26 2.01 mm to (50.2, 78.4)
- moved D49 2.01 mm to (17.8, 115.2)
- moved D54 2.01 mm to (122.9, 135.2)
- moved SW28 2.01 mm to (89.0, 76.6)
- moved SW31 2.01 mm to (177.2, 86.6)
- moved SW51 2.01 mm to (63.8, 118.7)
- moved SW50 2.01 mm to (44.9, 116.1)
- moved D24 2.01 mm to (261.7, 60.8)
- moved D4 2.01 mm to (86.0, 40.6)
- moved SW10 2.01 mm to (228.2, 38.6)
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Connections:
- D1 pad 1: unconnected-(D1-K-Pad1) -> Net-(D1-K)
- D10 pad 1: unconnected-(D10-K-Pad1) -> Net-(D1-K)
- D11 pad 1: unconnected-(D11-K-Pad1) -> Net-(D1-K)
- D12 pad 1: unconnected-(D12-K-Pad1) -> Net-(D1-K)
- D13 pad 1: unconnected-(D13-K-Pad1) -> Net-(D13-K)
- D14 pad 1: unconnected-(D14-K-Pad1) -> Net-(D13-K)
- D15 pad 1: unconnected-(D15-K-Pad1) -> Net-(D13-K)
- D16 pad 1: unconnected-(D16-K-Pad1) -> Net-(D13-K)
- D17 pad 1: unconnected-(D17-K-Pad1) -> Net-(D13-K)
- D18 pad 1: unconnected-(D18-K-Pad1) -> Net-(D13-K)
- D19 pad 1: unconnected-(D19-K-Pad1) -> Net-(D13-K)
- D2 pad 1: unconnected-(D2-K-Pad1) -> Net-(D1-K)
- D20 pad 1: unconnected-(D20-K-Pad1) -> Net-(D13-K)
- D21 pad 1: unconnected-(D21-K-Pad1) -> Net-(D13-K)
- D22 pad 1: unconnected-(D22-K-Pad1) -> Net-(D13-K)
- D23 pad 1: unconnected-(D23-K-Pad1) -> Net-(D13-K)
- D24 pad 1: unconnected-(D24-K-Pad1) -> Net-(D13-K)
- D25 pad 1: unconnected-(D25-K-Pad1) -> Net-(D25-K)
- D26 pad 1: unconnected-(D26-K-Pad1) -> Net-(D25-K)
- D27 pad 1: unconnected-(D27-K-Pad1) -> Net-(D25-K)
- D28 pad 1: unconnected-(D28-K-Pad1) -> Net-(D25-K)
- D29 pad 1: unconnected-(D29-K-Pad1) -> Net-(D25-K)
- D3 pad 1: unconnected-(D3-K-Pad1) -> Net-(D1-K)
- D30 pad 1: unconnected-(D30-K-Pad1) -> Net-(D25-K)
- D31 pad 1: unconnected-(D31-K-Pad1) -> Net-(D25-K)
- D32 pad 1: unconnected-(D32-K-Pad1) -> Net-(D25-K)
- D33 pad 1: unconnected-(D33-K-Pad1) -> Net-(D25-K)
- D34 pad 1: unconnected-(D34-K-Pad1) -> Net-(D25-K)
- D35 pad 1: unconnected-(D35-K-Pad1) -> Net-(D25-K)
- D36 pad 1: unconnected-(D36-K-Pad1) -> Net-(D25-K)
- D37 pad 1: unconnected-(D37-K-Pad1) -> Net-(D37-K)
- D38 pad 1: unconnected-(D38-K-Pad1) -> Net-(D37-K)
- D39 pad 1: unconnected-(D39-K-Pad1) -> Net-(D37-K)
- D4 pad 1: unconnected-(D4-K-Pad1) -> Net-(D1-K)
- D40 pad 1: unconnected-(D40-K-Pad1) -> Net-(D37-K)
- D41 pad 1: unconnected-(D41-K-Pad1) -> Net-(D37-K)
- D42 pad 1: unconnected-(D42-K-Pad1) -> Net-(D37-K)
- D43 pad 1: unconnected-(D43-K-Pad1) -> Net-(D37-K)
- D44 pad 1: unconnected-(D44-K-Pad1) -> Net-(D37-K)
- D45 pad 1: unconnected-(D45-K-Pad1) -> Net-(D37-K)
- D46 pad 1: unconnected-(D46-K-Pad1) -> Net-(D37-K)
- D47 pad 1: unconnected-(D47-K-Pad1) -> Net-(D37-K)
- D48 pad 1: unconnected-(D48-K-Pad1) -> Net-(D37-K)
- D49 pad 1: unconnected-(D49-K-Pad1) -> Net-(D49-K)
- D5 pad 1: unconnected-(D5-K-Pad1) -> Net-(D1-K)
- D50 pad 1: unconnected-(D50-K-Pad1) -> Net-(D49-K)
- D51 pad 1: unconnected-(D51-K-Pad1) -> Net-(D49-K)
- D52 pad 1: unconnected-(D52-K-Pad1) -> Net-(D49-K)
- D53 pad 1: unconnected-(D53-K-Pad1) -> Net-(D49-K)
- D54 pad 1: unconnected-(D54-K-Pad1) -> Net-(D49-K)
- D55 pad 1: unconnected-(D55-K-Pad1) -> Net-(D49-K)
- D56 pad 1: unconnected-(D56-K-Pad1) -> Net-(D49-K)
- D57 pad 1: unconnected-(D57-K-Pad1) -> Net-(D49-K)
- D58 pad 1: unconnected-(D58-K-Pad1) -> Net-(D49-K)
- D59 pad 1: unconnected-(D59-K-Pad1) -> Net-(D49-K)
- D6 pad 1: unconnected-(D6-K-Pad1) -> Net-(D1-K)
- D60 pad 1: unconnected-(D60-K-Pad1) -> Net-(D49-K)
- D7 pad 1: unconnected-(D7-K-Pad1) -> Net-(D1-K)
- D8 pad 1: unconnected-(D8-K-Pad1) -> Net-(D1-K)
- D9 pad 1: unconnected-(D9-K-Pad1) -> Net-(D1-K)
- SW1 pad 2: unconnected-(SW1-Pad2) -> Net-(SW1-Pad2)
- SW10 pad 2: unconnected-(SW10-Pad2) -> Net-(SW10-Pad2)
- SW11 pad 2: unconnected-(SW11-Pad2) -> Net-(SW11-Pad2)
- SW12 pad 2: unconnected-(SW12-Pad2) -> Net-(SW12-Pad2)
- SW13 pad 2: unconnected-(SW13-Pad2) -> Net-(SW1-Pad2)
- SW14 pad 2: unconnected-(SW14-Pad2) -> Net-(SW14-Pad2)
- SW15 pad 2: unconnected-(SW15-Pad2) -> Net-(SW15-Pad2)
- SW16 pad 2: unconnected-(SW16-Pad2) -> Net-(SW16-Pad2)
- SW17 pad 2: unconnected-(SW17-Pad2) -> Net-(SW17-Pad2)
- SW18 pad 2: unconnected-(SW18-Pad2) -> Net-(SW18-Pad2)
- SW19 pad 2: unconnected-(SW19-Pad2) -> Net-(SW19-Pad2)
- SW2 pad 2: unconnected-(SW2-Pad2) -> Net-(SW14-Pad2)
- SW20 pad 2: unconnected-(SW20-Pad2) -> Net-(SW20-Pad2)
- SW21 pad 2: unconnected-(SW21-Pad2) -> Net-(SW21-Pad2)
- SW22 pad 2: unconnected-(SW22-Pad2) -> Net-(SW10-Pad2)
- SW23 pad 2: unconnected-(SW23-Pad2) -> Net-(SW11-Pad2)
- SW24 pad 2: unconnected-(SW24-Pad2) -> Net-(SW12-Pad2)
- SW25 pad 2: unconnected-(SW25-Pad2) -> Net-(SW1-Pad2)
- SW26 pad 2: unconnected-(SW26-Pad2) -> Net-(SW14-Pad2)
- SW27 pad 2: unconnected-(SW27-Pad2) -> Net-(SW15-Pad2)
- SW28 pad 2: unconnected-(SW28-Pad2) -> Net-(SW16-Pad2)
- SW29 pad 2: unconnected-(SW29-Pad2) -> Net-(SW17-Pad2)
- SW3 pad 2: unconnected-(SW3-Pad2) -> Net-(SW15-Pad2)
- SW30 pad 2: unconnected-(SW30-Pad2) -> Net-(SW18-Pad2)
- SW31 pad 2: unconnected-(SW31-Pad2) -> Net-(SW19-Pad2)
- SW32 pad 2: unconnected-(SW32-Pad2) -> Net-(SW20-Pad2)
- SW33 pad 2: unconnected-(SW33-Pad2) -> Net-(SW21-Pad2)
- SW34 pad 2: unconnected-(SW34-Pad2) -> Net-(SW10-Pad2)
- SW35 pad 2: unconnected-(SW35-Pad2) -> Net-(SW11-Pad2)
- SW36 pad 2: unconnected-(SW36-Pad2) -> Net-(SW12-Pad2)
- SW37 pad 2: unconnected-(SW37-Pad2) -> Net-(SW1-Pad2)
- SW38 pad 2: unconnected-(SW38-Pad2) -> Net-(SW14-Pad2)
- SW39 pad 2: unconnected-(SW39-Pad2) -> Net-(SW15-Pad2)
- SW4 pad 2: unconnected-(SW4-Pad2) -> Net-(SW16-Pad2)
- SW40 pad 2: unconnected-(SW40-Pad2) -> Net-(SW16-Pad2)
- SW41 pad 2: unconnected-(SW41-Pad2) -> Net-(SW17-Pad2)
- SW42 pad 2: unconnected-(SW42-Pad2) -> Net-(SW18-Pad2)
- SW43 pad 2: unconnected-(SW43-Pad2) -> Net-(SW19-Pad2)
- SW44 pad 2: unconnected-(SW44-Pad2) -> Net-(SW20-Pad2)
- SW45 pad 2: unconnected-(SW45-Pad2) -> Net-(SW21-Pad2)
- SW46 pad 2: unconnected-(SW46-Pad2) -> Net-(SW10-Pad2)
- SW47 pad 2: unconnected-(SW47-Pad2) -> Net-(SW11-Pad2)
- SW48 pad 2: unconnected-(SW48-Pad2) -> Net-(SW12-Pad2)
- SW49 pad 2: unconnected-(SW49-Pad2) -> Net-(SW1-Pad2)
- SW5 pad 2: unconnected-(SW5-Pad2) -> Net-(SW17-Pad2)
- SW50 pad 2: unconnected-(SW50-Pad2) -> Net-(SW14-Pad2)
- SW51 pad 2: unconnected-(SW51-Pad2) -> Net-(SW15-Pad2)
- SW52 pad 2: unconnected-(SW52-Pad2) -> Net-(SW16-Pad2)
- SW53 pad 2: unconnected-(SW53-Pad2) -> Net-(SW17-Pad2)
- SW54 pad 2: unconnected-(SW54-Pad2) -> Net-(SW18-Pad2)
- SW55 pad 2: unconnected-(SW55-Pad2) -> Net-(SW19-Pad2)
- SW56 pad 2: unconnected-(SW56-Pad2) -> Net-(SW20-Pad2)
- SW57 pad 2: unconnected-(SW57-Pad2) -> Net-(SW21-Pad2)
- SW58 pad 2: unconnected-(SW58-Pad2) -> Net-(SW10-Pad2)
- SW59 pad 2: unconnected-(SW59-Pad2) -> Net-(SW11-Pad2)
- SW6 pad 2: unconnected-(SW6-Pad2) -> Net-(SW18-Pad2)
- SW60 pad 2: unconnected-(SW60-Pad2) -> Net-(SW12-Pad2)
- SW7 pad 2: unconnected-(SW7-Pad2) -> Net-(SW19-Pad2)
- SW8 pad 2: unconnected-(SW8-Pad2) -> Net-(SW20-Pad2)
- SW9 pad 2: unconnected-(SW9-Pad2) -> Net-(SW21-Pad2)
Routing:
- net Net-(D49-K): track 0.00 -> 263.0 mm
- net Net-(D25-K): track 0.00 -> 254.1 mm
- net Net-(D13-K): track 0.00 -> 248.8 mm
- net Net-(D1-K): track 0.00 -> 243.5 mm
- net Net-(D37-K): track 0.00 -> 200.4 mm
- net Net-(SW18-Pad2): track 0.00 -> 94.5 mm
- net Net-(SW19-Pad2): track 0.00 -> 92.6 mm
- net Net-(SW17-Pad2): track 0.00 -> 88.9 mm
- net Net-(SW20-Pad2): track 0.00 -> 87.9 mm
- net Net-(SW21-Pad2): track 0.00 -> 87.3 mm
- net Net-(SW16-Pad2): track 0.00 -> 87.3 mm
- net Net-(SW10-Pad2): track 0.00 -> 81.0 mm
- net Net-(SW15-Pad2): track 0.00 -> 81.0 mm
- net Net-(SW1-Pad2): track 0.00 -> 76.2 mm
- net Net-(SW14-Pad2): track 0.00 -> 76.2 mm
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
Commit message: Route the rows and cols to microcontroller
Parts:
- added SW61: SW_Push, marbastlib-mx:SW_MX_HS_CPG151101S11_1u, B.Cu at (79.0, 115.3)
- added SW62: SW_Push, marbastlib-mx:SW_MX_HS_CPG151101S11_1u, B.Cu at (216.9, 115.3)
- moved D52 12.8 mm to (95.9, 120.6)
- moved SW29 7.10 mm to (103.8, 75.5)
- moved D19 7.10 mm to (163.4, 65.7)
- moved SW40 7.10 mm to (82.7, 89.4)
- moved D54 7.10 mm to (119.3, 129.1)
- moved SW27 7.10 mm to (66.1, 70.2)
- moved D34 7.10 mm to (222.3, 74.2)
- moved D30 7.10 mm to (114.1, 82.3)
- moved D33 7.10 mm to (203.1, 74.5)
- moved D48 7.10 mm to (263.3, 92.5)
- moved SW34 7.10 mm to (229.8, 70.2)
- moved SW20 7.10 mm to (189.4, 56.6)
- moved SW45 7.10 mm to (213.3, 89.4)
- moved SW56 7.10 mm to (187.2, 121.7)
- moved SW10 7.10 mm to (224.5, 32.5)
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Connections:
- D1 pad 1: Net-(D1-K) -> row0
- D10 pad 1: Net-(D1-K) -> row0
- D11 pad 1: Net-(D1-K) -> row0
- D12 pad 1: Net-(D1-K) -> row0
- D13 pad 1: Net-(D13-K) -> row1
- D14 pad 1: Net-(D13-K) -> row1
- D15 pad 1: Net-(D13-K) -> row1
- D16 pad 1: Net-(D13-K) -> row1
- D17 pad 1: Net-(D13-K) -> row1
- D18 pad 1: Net-(D13-K) -> row1
- D19 pad 1: Net-(D13-K) -> row1
- D2 pad 1: Net-(D1-K) -> row0
- D20 pad 1: Net-(D13-K) -> row1
- D21 pad 1: Net-(D13-K) -> row1
- D22 pad 1: Net-(D13-K) -> row1
- D23 pad 1: Net-(D13-K) -> row1
- D24 pad 1: Net-(D13-K) -> row1
- D25 pad 1: Net-(D25-K) -> row2
- D26 pad 1: Net-(D25-K) -> row2
- D27 pad 1: Net-(D25-K) -> row2
- D28 pad 1: Net-(D25-K) -> row2
- D29 pad 1: Net-(D25-K) -> row2
- D3 pad 1: Net-(D1-K) -> row0
- D30 pad 1: Net-(D25-K) -> row2
- D31 pad 1: Net-(D25-K) -> row2
- D32 pad 1: Net-(D25-K) -> row2
- D33 pad 1: Net-(D25-K) -> row2
- D34 pad 1: Net-(D25-K) -> row2
- D35 pad 1: Net-(D25-K) -> row2
- D36 pad 1: Net-(D25-K) -> row2
- D37 pad 1: Net-(D37-K) -> row3
- D38 pad 1: Net-(D37-K) -> row3
- D39 pad 1: Net-(D37-K) -> row3
- D4 pad 1: Net-(D1-K) -> row0
- D40 pad 1: Net-(D37-K) -> row3
- D41 pad 1: Net-(D37-K) -> row3
- D42 pad 1: Net-(D37-K) -> row3
- D43 pad 1: Net-(D37-K) -> row3
- D44 pad 1: Net-(D37-K) -> row3
- D45 pad 1: Net-(D37-K) -> row3
- D46 pad 1: Net-(D37-K) -> row3
- D47 pad 1: Net-(D37-K) -> row3
- D48 pad 1: Net-(D37-K) -> row3
- D49 pad 1: Net-(D49-K) -> row4
- D5 pad 1: Net-(D1-K) -> row0
- D50 pad 1: Net-(D49-K) -> row4
- D51 pad 1: Net-(D49-K) -> row4
- D52 pad 1: Net-(D49-K) -> row4
- D53 pad 1: Net-(D49-K) -> row4
- D54 pad 1: Net-(D49-K) -> row4
- D55 pad 1: Net-(D49-K) -> row4
- D56 pad 1: Net-(D49-K) -> row4
- D57 pad 1: Net-(D49-K) -> row4
- D58 pad 1: Net-(D49-K) -> row4
- D59 pad 1: Net-(D49-K) -> row4
- D6 pad 1: Net-(D1-K) -> row0
- D60 pad 1: Net-(D49-K) -> row4
- D7 pad 1: Net-(D1-K) -> row0
- D8 pad 1: Net-(D1-K) -> row0
- D9 pad 1: Net-(D1-K) -> row0
- SW1 pad 2: Net-(SW1-Pad2) -> col0
- SW10 pad 2: Net-(SW10-Pad2) -> col9
- SW11 pad 2: Net-(SW11-Pad2) -> col10
- SW12 pad 2: Net-(SW12-Pad2) -> col11
- SW13 pad 2: Net-(SW1-Pad2) -> col0
- SW14 pad 2: Net-(SW14-Pad2) -> col1
- SW15 pad 2: Net-(SW15-Pad2) -> col2
- SW16 pad 2: Net-(SW16-Pad2) -> col3
- SW17 pad 2: Net-(SW17-Pad2) -> col4
- SW18 pad 2: Net-(SW18-Pad2) -> col5
- SW19 pad 2: Net-(SW19-Pad2) -> col6
- SW2 pad 2: Net-(SW14-Pad2) -> col1
- SW20 pad 2: Net-(SW20-Pad2) -> col7
- SW21 pad 2: Net-(SW21-Pad2) -> col8
- SW22 pad 2: Net-(SW10-Pad2) -> col9
- SW23 pad 2: Net-(SW11-Pad2) -> col10
- SW24 pad 2: Net-(SW12-Pad2) -> col11
- SW25 pad 2: Net-(SW1-Pad2) -> col0
- SW26 pad 2: Net-(SW14-Pad2) -> col1
- SW27 pad 2: Net-(SW15-Pad2) -> col2
- SW28 pad 2: Net-(SW16-Pad2) -> col3
- SW29 pad 2: Net-(SW17-Pad2) -> col4
- SW3 pad 2: Net-(SW15-Pad2) -> col2
- SW30 pad 2: Net-(SW18-Pad2) -> col5
- SW31 pad 2: Net-(SW19-Pad2) -> col6
- SW32 pad 2: Net-(SW20-Pad2) -> col7
- SW33 pad 2: Net-(SW21-Pad2) -> col8
- SW34 pad 2: Net-(SW10-Pad2) -> col9
- SW35 pad 2: Net-(SW11-Pad2) -> col10
- SW36 pad 2: Net-(SW12-Pad2) -> col11
- SW37 pad 2: Net-(SW1-Pad2) -> col0
- SW38 pad 2: Net-(SW14-Pad2) -> col1
- SW39 pad 2: Net-(SW15-Pad2) -> col2
- SW4 pad 2: Net-(SW16-Pad2) -> col3
- SW40 pad 2: Net-(SW16-Pad2) -> col3
- SW41 pad 2: Net-(SW17-Pad2) -> col4
- SW42 pad 2: Net-(SW18-Pad2) -> col5
- SW43 pad 2: Net-(SW19-Pad2) -> col6
- SW44 pad 2: Net-(SW20-Pad2) -> col7
- SW45 pad 2: Net-(SW21-Pad2) -> col8
- SW46 pad 2: Net-(SW10-Pad2) -> col9
- SW47 pad 2: Net-(SW11-Pad2) -> col10
- SW48 pad 2: Net-(SW12-Pad2) -> col11
- SW49 pad 2: Net-(SW1-Pad2) -> col0
- SW5 pad 2: Net-(SW17-Pad2) -> col4
- SW50 pad 2: Net-(SW14-Pad2) -> col1
- SW51 pad 2: Net-(SW15-Pad2) -> col2
- SW52 pad 1: Net-(D52-A) -> col3
- SW52 pad 2: Net-(SW16-Pad2) -> Net-(D52-A)
- SW53 pad 2: Net-(SW17-Pad2) -> col4
- SW54 pad 2: Net-(SW18-Pad2) -> col5
- SW55 pad 2: Net-(SW19-Pad2) -> col6
- SW56 pad 2: Net-(SW20-Pad2) -> col7
- SW57 pad 2: Net-(SW21-Pad2) -> col8
- SW58 pad 2: Net-(SW10-Pad2) -> col9
- SW59 pad 2: Net-(SW11-Pad2) -> col10
- SW6 pad 2: Net-(SW18-Pad2) -> col5
- SW60 pad 2: Net-(SW12-Pad2) -> col11
- SW7 pad 2: Net-(SW19-Pad2) -> col6
- SW8 pad 2: Net-(SW20-Pad2) -> col7
- SW9 pad 2: Net-(SW21-Pad2) -> col8
- U1 pad 11: unconnected-(U1-10-Pad11) -> row0
- U1 pad 12: unconnected-(U1-11-Pad12) -> row1
- U1 pad 13: unconnected-(U1-12-Pad13) -> row2
- U1 pad 14: unconnected-(U1-13-Pad14) -> row3
- U1 pad 15: unconnected-(U1-14-Pad15) -> col4
- U1 pad 16: unconnected-(U1-15-Pad16) -> col5
- U1 pad 17: unconnected-(U1-26-Pad17) -> col3
- U1 pad 18: unconnected-(U1-27-Pad18) -> col2
- U1 pad 19: unconnected-(U1-28-Pad19) -> col1
- U1 pad 20: unconnected-(U1-29-Pad20) -> col0
- U1 pad 3: unconnected-(U1-2-Pad3) -> row4
- U1 pad 4: unconnected-(U1-3-Pad4) -> col11
- U1 pad 5: unconnected-(U1-4-Pad5) -> col10
- U1 pad 6: unconnected-(U1-5-Pad6) -> col9
- U1 pad 7: unconnected-(U1-6-Pad7) -> col8
- U1 pad 8: unconnected-(U1-7-Pad8) -> col6
- U1 pad 9: unconnected-(U1-8-Pad9) -> col7
Routing:
- net row4: track 0.00 -> 298.7 mm
- net row0: track 0.00 -> 288.4 mm
- net row1: track 0.00 -> 274.8 mm, vias 0 -> 2
- net row3: track 0.00 -> 267.9 mm
- net Net-(D49-K): track 263.0 -> 0.00 mm
- net row2: track 0.00 -> 261.3 mm, vias 0 -> 2
- net Net-(D25-K): track 254.1 -> 0.00 mm
- net Net-(D13-K): track 248.8 -> 0.00 mm
- net Net-(D1-K): track 243.5 -> 0.00 mm
- net Net-(D37-K): track 200.4 -> 0.00 mm
- net col11: track 0.00 -> 198.9 mm, vias 0 -> 1
- net col0: track 0.00 -> 193.8 mm, vias 0 -> 1
- net col10: track 0.00 -> 180.1 mm, vias 0 -> 1
- net col1: track 0.00 -> 175.0 mm, vias 0 -> 1
- net col9: track 0.00 -> 166.0 mm, vias 0 -> 1
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
Commit message: Add rounded corners
Other:
- board size 272.6 x 122.9 mm -> 272.4 x 122.9 mm

Commit message: Update rp2040 tiny footprint
Parts:
- U1: footprint mcu:rp2040-zero-smd -> rp2040-tiny:rp2040-tiny
- moved D44 10.8 mm to (182.5, 88.6)
- moved D59 10.8 mm to (242.4, 104.2)
- moved D4 10.8 mm to (77.6, 24.8)
- moved D24 10.8 mm to (253.4, 45.0)
- moved SW22 10.8 mm to (222.5, 41.6)
- moved SW16 10.8 mm to (83.3, 41.9)
- moved D9 10.8 mm to (193.1, 27.0)
- moved D38 10.8 mm to (30.9, 83.2)
- moved SW42 10.8 mm to (115.0, 89.6)
- moved D39 10.8 mm to (50.5, 81.1)
- moved D14 10.8 mm to (36.2, 45.4)
- moved SW47 10.8 mm to (247.3, 81.4)
- moved SW33 10.8 mm to (205.9, 60.7)
- moved SW6 10.8 mm to (123.0, 33.0)
- moved D1 10.8 mm to (20.0, 23.9)
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Routing:
- net row3: track 267.9 -> 269.9 mm
- net row1: track 274.8 -> 273.2 mm
- net row2: track 261.3 -> 259.7 mm
- net row0: track 288.4 -> 286.8 mm
- net col3: track 159.6 -> 158.1 mm
- net col2: track 160.9 -> 159.4 mm
- net col9: track 166.0 -> 164.5 mm
- net col11: track 198.9 -> 197.5 mm
- net col1: track 175.0 -> 173.5 mm
- net col10: track 180.1 -> 178.6 mm
- net col8: track 162.4 -> 160.9 mm
- net col0: track 193.8 -> 192.4 mm
- net col6: track 115.2 -> 114.0 mm
- net col5: track 108.5 -> 107.3 mm
- net col4: track 121.5 -> 120.3 mm
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