File: src/pcb/form-uno/form-uno.kicad_sch (KiCad schematic)
At the start: 123 parts, among them SW1 SW_Push, SW10 SW_Push, SW11 SW_Push, SW12 SW_Push, SW13 SW_Push, SW14 SW_Push, SW15 SW_Push, SW16 SW_Push, SW17 SW_Push, SW18 SW_Push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

Commit message: Set pcb revision
Other:
- title: (none) -> Form Uno
Changed lines of the file:
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@@
 	(generator_version "8.0")
 	(paper "A4")
+	(title_block
+		(title "Form Uno")
+		(date "2024-07-29")
+		(rev "1.0")
+	)
 	(junction
 		(at 162.56 102.87)
